File: PCB/Gabi/HUB/HUB.kicad_sch (KiCad schematic)
At the start: 18 parts

Commit message: oui
Parts:
- J2: renamed from J?; footprint (none) -> Connector_USB:USB_C_Plug_Molex_105444
- gave numbers to parts that had none: 17
